File: hardware/sensorpcb.sch (KiCad schematic (older format))
At the start: 8 parts, among them P1 CONN_01X02

Commit message: added decoupling capacitor to schematic
Parts:
- added C2: 100nF, symbol C
Connections:
- wire segments 30 -> 32
Other:
- note added: "Decoupling\nCapacitor - \nplace close\nto ESP-01"
- moved on the sheet: C1, ESP1, P1
Changed lines of the file:
@@
 L ESP-01 ESP1
 U 1 1 55FFE6A1
-P 2100 1100
-F 0 "ESP1" H 2100 1400 60  0000 C CNN
-F 1 "ESP-01" H 2100 800 60  0000 C CNN
-F 2 "" H 1900 1000 60  0000 C CNN
-F 3 "" H 1900 1000 60  0000 C CNN
-	1    2100 1100
+P 1700 1100
+F 0 "ESP1" H 1700 1400 60  0000 C CNN
+F 1 "ESP-01" H 1700 800 60  0000 C CNN
+F 2 "" H 1500 1000 60  0000 C CNN
+F 3 "" H 1500 1000 60  0000 C CNN
+	1    1700 1100
 	1    0    0    -1
 $EndComp
@@
 L +3.3V #PWR01
 U 1 1 55FFEB33
-P 1900 2050
-F 0 "#PWR01" H 1900 1900 50  0001 C CNN
-F 1 "+3.3V" H 1900 2190 50  0000 C CNN
-F 2 "" H 1900 2050 60  0000 C CNN
-F 3 "" H 1900 2050 60  0000 C CNN
-	1    1900 2050
+P 1250 2050
+F 0 "#PWR01" H 1250 1900 50  0001 C CNN
+F 1 "+3.3V" H 1250 2190 50  0000 C CNN
+F 2 "" H 1250 2050 60  0000 C CNN
+F 3 "" H 1250 2050 60  0000 C CNN
+	1    1250 2050
 	1    0    0    -1
 $EndComp
@@
 L GNDREF #PWR02
 U 1 1 55FFEB54
-P 1900 2550
-F 0 "#PWR02" H 1900 2300 50  0001 C CNN
-F 1 "GNDREF" H 1900 2400 50  0000 C CNN
-F 2 "" H 1900 2550 60  0000 C CNN
-F 3 "" H 1900 2550 60  0000 C CNN
-	1    1900 2550
-	1    0    0    -1
-$EndComp
-Text GLabel 1750 2100 0    60   UnSpc ~ 0
-3V3
-Text GLabel 1750 2500 0    60   UnSpc ~ 0
-GND
-Text GLabel 3050 1150 2    60   Input ~ 0
+P 1250 2550
+F 0 "#PWR02" H 1250 2300 50  0001 C CNN
+F 1 "GNDREF" H 1250 2400 50  0000 C CNN
+F 2 "" H 1250 2550 60  0000 C CNN
+F 3 "" H 1250 2550 60  0000 C CNN
+	1    1250 2550
+	1    0    0    -1
+$EndComp
+Text GLabel 1100 2100 0    60   UnSpc ~ 0
+3V3
+Text GLabel 1100 2500 0    60   UnSpc ~ 0
+GND
+Text GLabel 2650 1150 2    60   Input ~ 0
 SENSOR-DATA
 Text GLabel 5500 1100 2    60   Output ~ 0
@@
 Text GLabel 5500 950  2    60   UnSpc ~ 0
 GND
-Text GLabel 3050 950  2    60   UnSpc ~ 0
-GND
-Text GLabel 3050 1550 2    60   UnSpc ~ 0
+Text GLabel 2650 950  2    60   UnSpc ~ 0
+GND
+Text GLabel 2650 1550 2    60   UnSpc ~ 0
 3V3
 $Comp
 L CP C1
 U 1 1 55FFECDB
-P 1900 2300
-F 0 "C1" H 1925 2400 50  0000 L CNN
-F 1 "100uF" H 1925 2200 50  0000 L CNN
-F 2 "" H 1938 2150 30  0000 C CNN
-F 3 "" H 1900 2300 60  0000 C CNN
-	1    1900 2300
-	1    0    0    -1
-$EndComp
-NoConn ~ 2600 1250
-NoConn ~ 1550 950
+P 1250 2300
+F 0 "C1" H 1275 2400 50  0000 L CNN
+F 1 "100uF" H 1275 2200 50  0000 L CNN
+F 2 "" H 1288 2150 30  0000 C CNN
+F 3 "" H 1250 2300 60  0000 C CNN
+	1    1250 2300
+	1    0    0    -1
+$EndComp
+NoConn ~ 2200 1250
+NoConn ~ 1150 950
 $Comp
 L R R1
 U 1 1 55FFEFC8
-P 1200 1300
-F 0 "R1" V 1280 1300 50  0000 C CNN
-F 1 "10k" V 1200 1300 50  0000 C CNN
-F 2 "" V 1130 1300 30  0000 C CNN
-F 3 "" H 1200 1300 30  0000 C CNN
-	1    1200 1300
+P 800 1300
+F 0 "R1" V 880 1300 50  0000 C CNN
+F 1 "10k" V 800 1300 50  0000 C CNN
+F 2 "" V 730 1300 30  0000 C CNN
+F 3 "" H 800 1300 30  0000 C CNN
+	1    800  1300
 	1    0    0    -1
 $EndComp
@@
 L R R2
 U 1 1 55FFF00F
-P 1400 1300
-F 0 "R2" V 1480 1300 50  0000 C CNN
-F 1 "10k" V 1400 1300 50  0000 C CNN
-F 2 "" V 1330 1300 30  0000 C CNN
-F 3 "" H 1400 1300 30  0000 C CNN
-	1    1400 1300
+P 1000 1300
+F 0 "R2" V 1080 1300 50  0000 C CNN
+F 1 "10k" V 1000 1300 50  0000 C CNN
+F 2 "" V 930 1300 30  0000 C CNN
+F 3 "" H 1000 1300 30  0000 C CNN
+	1    1000 1300
 	1    0    0    -1
 $EndComp
@@
 L R R3
 U 1 1 55FFF172
-P 2900 1300
-F 0 "R3" V 2980 1300 50  0000 C CNN
-F 1 "10k" V 2900 1300 50  0000 C CNN
-F 2 "" V 2830 1300 30  0000 C CNN
-F 3 "" H 2900 1300 30  0000 C CNN
-	1    2900 1300
-	1    0    0    -1
-$EndComp
-NoConn ~ 2600 1150
+P 2500 1300
+F 0 "R3" V 2580 1300 50  0000 C CNN
+F 1 "10k" V 2500 1300 50  0000 C CNN
+F 2 "" V 2430 1300 30  0000 C CNN
+F 3 "" H 2500 1300 30  0000 C CNN
+	1    2500 1300
+	1    0    0    -1
+$EndComp
+NoConn ~ 2200 1150
 $Comp
 L CONN_01X02 P1
 U 1 1 55FFFB03
-P 2600 2300
-F 0 "P1" H 2600 2450 50  0000 C CNN
-F 1 "CONN_01X02" V 2700 2300 50  0000 C CNN
-F 2 "" H 2600 2300 60  0000 C CNN
-F 3 "" H 2600 2300 60  0000 C CNN
-	1    2600 2300
+P 1950 2300
+F 0 "P1" H 1950 2450 50  0000 C CNN
+F 1 "CONN_01X02" V 2050 2300 50  0000 C CNN
+F 2 "" H 1950 2300 60  0000 C CNN
+F 3 "" H 1950 2300 60  0000 C CNN
+	1    1950 2300
 	1    0    0    -1
 $EndComp
@@
 L PWR_FLAG #FLG03
 U 1 1 55FFFDCE
-P 2300 2100
-F 0 "#FLG03" H 2300 2195 50  0001 C CNN
-F 1 "PWR_FLAG" H 2300 2280 50  0000 C CNN
-F 2 "" H 2300 2100 60  0000 C CNN
-F 3 "" H 2300 2100 60  0000 C CNN
-	1    2300 2100
+P 1650 2100
+F 0 "#FLG03" H 1650 2195 50  0001 C CNN
+F 1 "PWR_FLAG" H 1650 2280 50  0000 C CNN
+F 2 "" H 1650 2100 60  0000 C CNN
+F 3 "" H 1650 2100 60  0000 C CNN
+	1    1650 2100
 	1    0    0    -1
 $EndComp
@@
 L PWR_FLAG #FLG04
 U 1 1 55FFFE05
-P 2300 2500
-F 0 "#FLG04" H 2300 2595 50  0001 C CNN
-F 1 "PWR_FLAG" H 2300 2680 50  0000 C CNN
-F 2 "" H 2300 2500 60  0000 C CNN
-F 3 "" H 2300 2500 60  0000 C CNN
-	1    2300 2500
+P 1650 2500
+F 0 "#FLG04" H 1650 2595 50  0001 C CNN
+F 1 "PWR_FLAG" H 1650 2680 50  0000 C CNN
+F 2 "" H 1650 2500 60  0000 C CNN
+F 3 "" H 1650 2500 60  0000 C CNN
+	1    1650 2500
 	-1   0    0    1
 $EndComp
@@
 SENSOR-DATA
 Wire Wire Line
-	1550 1550 1550 1250
-Wire Wire Line
-	1200 1550 3050 1550
-Wire Wire Line
-	2900 1150 2900 1050
-Wire Wire Line
-	2900 1550 2900 1450
-Wire Wire Line
-	1900 2450 1900 2550
-Wire Wire Line
-	1900 2050 1900 2150
-Wire Wire Line
-	1750 2100 2400 2100
-Connection ~ 1900 2100
-Wire Wire Line
-	1750 2500 2400 2500
-Connection ~ 1900 2500
-Wire Wire Line
-	2400 2100 2400 2250
-Wire Wire Line
-	2400 2500 2400 2350
-Connection ~ 2300 2100
-Connection ~ 2300 2500
-Wire Wire Line
-	1200 1150 1200 1050
-Wire Wire Line
-	1200 1050 1550 1050
-Wire Wire Line
-	1400 1150 1550 1150
-Wire Wire Line
-	1200 1450 1200 1550
-Connection ~ 1550 1550
-Wire Wire Line
-	1400 1450 1400 1550
-Connection ~ 1400 1550
-Connection ~ 2900 1550
-Wire Wire Line
-	2900 1050 2600 1050
-Wire Wire Line
-	2900 1150 3050 1150
-Connection ~ 2900 1150
-Wire Wire Line
-	2600 950  3050 950
+	1150 1550 1150 1250
+Wire Wire Line
+	800  1550 2650 1550
+Wire Wire Line
+	2500 1150 2500 1050
+Wire Wire Line
+	2500 1550 2500 1450
+Wire Wire Line
+	1250 2450 1250 2550
+Wire Wire Line
+	1250 2050 1250 2150
+Wire Wire Line
+	1100 2100 1750 2100
+Connection ~ 1250 2100
+Wire Wire Line
+	1100 2500 1750 2500
+Connection ~ 1250 2500
+Wire Wire Line
+	1750 2100 1750 2250
+Wire Wire Line
+	1750 2500 1750 2350
+Connection ~ 1650 2100
+Connection ~ 1650 2500
+Wire Wire Line
+	800  1150 800  1050
+Wire Wire Line
+	800  1050 1150 1050
+Wire Wire Line
+	1000 1150 1150 1150
+Wire Wire Line
+	800  1450 800  1550
+Connection ~ 1150 1550
+Wire Wire Line
+	1000 1450 1000 1550
+Connection ~ 1000 1550
+Connection ~ 2500 1550
+Wire Wire Line
+	2500 1050 2200 1050
+Wire Wire Line
+	2500 1150 2650 1150
+Connection ~ 2500 1150
+Wire Wire Line
+	2200 950  2650 950
 Wire Wire Line
 	5350 950  5500 950
@@
 Wire Wire Line
 	5400 2400 5550 2400
-Text Notes 4350 1900 0    60   ~ 0
+Text Notes 4600 1850 0    60   ~ 0
 Populate either the DS18S20 temperature sensor\nor the DHT22 temperature/humidity sensor, but \nnot both!
+$Comp
+L C C2
+U 1 1 5605B759
+P 3000 2250
+F 0 "C2" H 3025 2350 50  0000 L CNN
+F 1 "100nF" H 3025 2150 50  0000 L CNN
+F 2 "" H 3038 2100 30  0000 C CNN
+F 3 "" H 3000 2250 60  0000 C CNN
+	1    3000 2250
+	1    0    0    -1
+$EndComp
+Text GLabel 3000 2000 1    60   UnSpc ~ 0
+GND
+Text GLabel 3000 2500 3    60   UnSpc ~ 0
+3V3
+Wire Wire Line
+	3000 2400 3000 2500
+Wire Wire Line
+	3000 2000 3000 2100
+Text Notes 3300 2450 0    60   ~ 0
+Decoupling\nCapacitor - \nplace close\nto ESP-01
 $EndSCHEMATC

Commit message: added esp-wroom-02 to schematic
Parts:
- added R4, R5, R6, R7, R8: 10k, symbol R-RESCUE-sensorpcb
- added WROOM-02-1: ESP8266_WROOM_02, symbol ESP8266_WROOM_02
- C2: symbol C -> C-RESCUE-sensorpcb
- R1, R2, R3: symbol R -> R-RESCUE-sensorpcb
Connections:
- wire segments 32 -> 50
- no-connect marks 4 -> 13
Other:
- moved on the sheet: C1, DHT221, DS18S20-1, ESP1, P1

Commit message: updated schematic for website
Parts:
- C1: symbol CP -> CP-RESCUE-sensorpcb
Connections:
- wire segments 50 -> 62
Other:
- note added: "Populate either the ESP1 or \nthe ESP-WROOM-02 but \nnot both!"
- moved on the sheet: DHT221, DS18S20-1, ESP1, R1, R2, R3, R4, R5, R6, R7, R8, WROOM-02-1
